File: Single_transistor_AMP/Single_transistor_AMP.sch (KiCad schematic (older format))
At the start: 10 parts, among them J1 Conn_01x02, J2 Conn_01x02, Q1 2N2219

Commit message: first commit
Parts:
- C1, C2: footprint Capacitor_Tantalum_SMD:CP_EIA-1608-08_AVX-J -> Capacitor_THT:C_Disc_D4.7mm_W2.5mm_P5.00mm
- C3: value 20uF -> 22uF; footprint Capacitor_Tantalum_SMD:CP_EIA-1608-08_AVX-J -> Capacitor_THT:C_Disc_D4.7mm_W2.5mm_P5.00mm
- J1, J2: footprint Connector:Banana_Jack_2Pin -> TerminalBlock:TerminalBlock_Altech_AK300-2_P5.00mm
- R1, R2, R3, R4: footprint Resistor_SMD:R_1806_4516Metric_Pad1.57x1.80mm_HandSolder -> Resistor_THT:R_Axial_DIN0204_L3.6mm_D1.6mm_P7.62mm_Horizontal
Changed lines of the file:
@@
 F 0 "J1" H 1470 3425 50  0000 C CNN
 F 1 "Conn_01x02" H 1470 3516 50  0000 C CNN
-F 2 "Connector:Banana_Jack_2Pin" H 1550 3750 50  0001 C CNN
+F 2 "TerminalBlock:TerminalBlock_Altech_AK300-2_P5.00mm" H 1550 3750 50  0001 C CNN
 F 3 "https://media.digikey.com/pdf/Data%20Sheets/Phoenix%20Contact%20PDFs/5442895.pdf" H 1550 3750 50  0001 C CNN
 	1    1550 3750
@@
 F 0 "C1" V 2398 3650 50  0000 C CNN
 F 1 "1uF" V 2489 3650 50  0000 C CNN
-F 2 "Capacitor_Tantalum_SMD:CP_EIA-1608-08_AVX-J" H 2688 3500 50  0001 C CNN
-F 3 "https://eu.mouser.com/datasheet/2/212/KEM_C1092_GOLDMAX_X8R-1101978.pdf" H 2650 3650 50  0001 C CNN
+F 2 "Capacitor_THT:C_Disc_D4.7mm_W2.5mm_P5.00mm" H 2688 3500 50  0001 C CNN
+F 3 "https://eu.mouser.com/datasheet/2/281/c49e-506.pdf" H 2650 3650 50  0001 C CNN
 	1    2650 3650
 	0    1    1    0
@@
 F 0 "R1" H 3570 4196 50  0000 L CNN
 F 1 "1K" H 3570 4105 50  0000 L CNN
-F 2 "Resistor_SMD:R_1806_4516Metric_Pad1.57x1.80mm_HandSolder" V 3430 4150 50  0001 C CNN
+F 2 "Resistor_THT:R_Axial_DIN0204_L3.6mm_D1.6mm_P7.62mm_Horizontal" V 3430 4150 50  0001 C CNN
 F 3 "https://eu.mouser.com/datasheet/2/447/Yageo%20LR_CFR_2013-595289.pdf" H 3500 4150 50  0001 C CNN
 	1    3500 4150
@@
 F 0 "R2" H 3570 3246 50  0000 L CNN
 F 1 "4.7K" H 3570 3155 50  0000 L CNN
-F 2 "Resistor_SMD:R_1806_4516Metric_Pad1.57x1.80mm_HandSolder" V 3430 3200 50  0001 C CNN
+F 2 "Resistor_THT:R_Axial_DIN0204_L3.6mm_D1.6mm_P7.62mm_Horizontal" V 3430 3200 50  0001 C CNN
 F 3 "https://eu.mouser.com/datasheet/2/219/CF-6922.pdf" H 3500 3200 50  0001 C CNN
 	1    3500 3200
@@
 F 0 "R3" H 4770 3246 50  0000 L CNN
 F 1 "4.7K" H 4770 3155 50  0000 L CNN
-F 2 "Resistor_SMD:R_1806_4516Metric_Pad1.57x1.80mm_HandSolder" V 4630 3200 50  0001 C CNN
+F 2 "Resistor_THT:R_Axial_DIN0204_L3.6mm_D1.6mm_P7.62mm_Horizontal" V 4630 3200 50  0001 C CNN
 F 3 "https://eu.mouser.com/datasheet/2/219/CF-6922.pdf" H 4700 3200 50  0001 C CNN
 	1    4700 3200
@@
 F 0 "R4" H 4770 4196 50  0000 L CNN
 F 1 "1K" H 4770 4105 50  0000 L CNN
-F 2 "Resistor_SMD:R_1806_4516Metric_Pad1.57x1.80mm_HandSolder" V 4630 4150 50  0001 C CNN
+F 2 "Resistor_THT:R_Axial_DIN0204_L3.6mm_D1.6mm_P7.62mm_Horizontal" V 4630 4150 50  0001 C CNN
 F 3 "https://eu.mouser.com/datasheet/2/447/Yageo%20LR_CFR_2013-595289.pdf" H 4700 4150 50  0001 C CNN
 	1    4700 4150
@@
 P 5400 4150
 F 0 "C3" H 5515 4196 50  0000 L CNN
-F 1 "20uF" H 5515 4105 50  0000 L CNN
-F 2 "Capacitor_Tantalum_SMD:CP_EIA-1608-08_AVX-J" H 5438 4000 50  0001 C CNN
-F 3 "~" H 5400 4150 50  0001 C CNN
+F 1 "22uF" H 5515 4105 50  0000 L CNN
+F 2 "Capacitor_THT:C_Disc_D4.7mm_W2.5mm_P5.00mm" H 5438 4000 50  0001 C CNN
+F 3 "http://www.vishay.com/docs/23118/564r565r.pdf" H 5400 4150 50  0001 C CNN
 	1    5400 4150
 	1    0    0    -1
@@
 F 0 "C2" V 5048 3450 50  0000 C CNN
 F 1 "4.7uF" V 5139 3450 50  0000 C CNN
-F 2 "Capacitor_Tantalum_SMD:CP_EIA-1608-08_AVX-J" H 5338 3300 50  0001 C CNN
+F 2 "Capacitor_THT:C_Disc_D4.7mm_W2.5mm_P5.00mm" H 5338 3300 50  0001 C CNN
 F 3 "https://eu.mouser.com/datasheet/2/281/Murata%20RPE%20Series-202940.pdf" H 5300 3450 50  0001 C CNN
 	1    5300 3450
@@
 F 0 "J2" H 6480 3442 50  0000 L CNN
 F 1 "Conn_01x02" H 6480 3351 50  0000 L CNN
-F 2 "Connector:Banana_Jack_2Pin" H 6400 3450 50  0001 C CNN
+F 2 "TerminalBlock:TerminalBlock_Altech_AK300-2_P5.00mm" H 6400 3450 50  0001 C CNN
 F 3 "https://media.digikey.com/pdf/Data%20Sheets/Phoenix%20Contact%20PDFs/5442895.pdf" H 6400 3450 50  0001 C CNN
 	1    6400 3450
@@
 F 1 "VCC" H 5517 3173 50  0000 C CNN
 F 2 "Connector_Pin:Pin_D0.7mm_L6.5mm_W1.8mm_FlatFork" H 5500 3000 50  0001 C CNN
-F 3 "" H 5500 3000 50  0001 C CNN
+F 3 "https://cdn.harwin.com/pdfs/M20-782.pdf" H 5500 3000 50  0001 C CNN
 	1    5500 3000
 	1    0    0    -1
